Commit message: Added Limits to Joints

File: description/robot_core.xacro (robot description, xacro)
@@ -99,9 +99,10 @@
     </link>
     <!-- Hinge at the Pin -->
-    <joint name="pin_hinge_joint" type="continuous">
+    <joint name="pin_hinge_joint" type="revolute">
         <parent link="pillar_connecting_link"/>
         <child link="pin_hinge_link"/>
         <origin xyz="0.0 0.0 0.0" rpy="0.0 0.0 ${pi/2}"/>
         <axis xyz="0.0 0.0 1"/>
+        <limit lower="-0.39" upper="0.39" effort="0.0" velocity="0.0"/>
     </joint>
     <link name="pin_hinge_link">
@@ -126,5 +127,5 @@
                 <box size="0.012 0.55 0.012"/>
             </geometry>
-            <material name="white"/>
+            <material name="black"/>
         </visual>
     </link>
