Commit message: Added Bldc motor base

File: description/robot.urdf.xacro (robot description, xacro)
@@ -3,3 +3,4 @@
     <!-- Example link -->
     <xacro:include filename="robot_core.xacro"/>
+    <xacro:include filename="bldc_motor.xacro"/>
 </robot>

File: description/robot_core.xacro (robot description, xacro)
@@ -6,4 +6,7 @@
     <material name="black">
         <color rgba="0.0 0.0 0.0 1.0"/>
+    </material>
+    <material name="gray">
+        <color rgba="0.5 0.5 0.5 1.0"/>
     </material>
     <link name="base_link">
