Commit message: Added Rotors to Motors

File: description/bldc_motor.xacro (robot description, xacro)
@@ -21,5 +21,5 @@
                 <cylinder radius="0.02" length="0.01"/>
             </geometry>
-            <origin xyz="0.0 0.0 0.0" rpy="0.0 0.0 0.0"/>
+            <origin xyz="0.0 0.0 0.0" rpy="0.0 ${pi} 0.0"/>
             <material name="gray"/>
         </visual>
@@ -44,3 +44,49 @@
         <origin xyz="0.01 -0.25 0.0" rpy="0.0 ${pi/2} 0.0"/>
     </joint>
+    <!-- Rotors for BLDC  -->
+    <link name="rotor_L">
+        <visual>
+            <geometry>
+                <cylinder radius="0.12" length="0.001"/>
+            </geometry>
+            <origin xyz="0.0 0.0 0.0" rpy="0.0 0.0 0.0"/>
+            <material name="blue"/>
+        </visual>
+    </link>
+    <joint name="rotor_l_joint" type="continuous">
+        <parent link="base_link_motor_b_L"/>
+        <child link="rotor_L"/>
+        <origin xyz="0.0 0.0 0.005" rpy="0.0 0.0 0.0"/>
+        <axis xyz="0.0 0.0 1.0"/>
+    </joint>
+    <link name="rotor_R">
+        <visual>
+            <geometry>
+                <cylinder radius="0.12" length="0.001"/>
+            </geometry>
+            <origin xyz="0.0 0.0 0.0" rpy="0.0 0.0 0.0"/>
+            <material name="blue"/>
+        </visual>
+    </link>
+    <joint name="rotor_r_joint" type="continuous">
+        <parent link="base_link_motor_b_R"/>
+        <child link="rotor_R"/>
+        <origin xyz="0.0 0.0 -0.005" rpy="0.0 0.0 0.0"/>
+        <axis xyz="0.0 0.0 1.0"/>
+    </joint>
+    <link name="rotor_pitch">
+        <visual>
+            <geometry>
+                <cylinder radius="0.12" length="0.001"/>
+            </geometry>
+            <origin xyz="0.0 0.0 0.0" rpy="0.0 0.0 0.0"/>
+            <material name="blue"/>
+        </visual>
+    </link>
+    <joint name="rotor_pitch_joint" type="continuous">
+        <parent link="base_link_motor_pitch"/>
+        <child link="rotor_pitch"/>
+        <origin xyz="0.0 0.0 0.005" rpy="0.0 0.0 0.0"/>
+        <axis xyz="0.0 0.0 1.0"/>
+    </joint>
 </robot>

File: description/robot_core.xacro (robot description, xacro)
@@ -9,4 +9,7 @@
     <material name="gray">
         <color rgba="0.5 0.5 0.5 1.0"/>
+    </material>
+    <material name="blue">
+        <color rgba="0.0 0.0 1.0 0.5"/>
     </material>
     <link name="base_link">

Commit message: Gazebo camera plugin added

File: description/bldc_motor.xacro (robot description, xacro)
@@ -1,4 +1,5 @@
 <?xml version="1.0"?>
 <robot xmlns:xacro="http://www.ros.org/wiki/xacro" name="bldc_motor">
+    <xacro:include filename="inertial_macros.xacro"/>
     <!-- Bldc Motors Base -->
     <link name="base_link_motor_b_L">
@@ -10,4 +11,12 @@
             <material name="gray"/>
         </visual>
+        <collision>
+            <geometry>
+                <cylinder radius="0.02" length="0.01"/>
+            </geometry>
+        </collision>
+        <xacro:inertial_cylinder mass= "0.06" radius="0.02" length="0.01">
+            <origin xyz="0 0 0" rpy="0 0 0"/>
+        </xacro:inertial_cylinder>
     </link>
     <joint name="base_joint_b_L" type="fixed">
@@ -24,4 +33,12 @@
             <material name="gray"/>
         </visual>
+        <collision>
+            <geometry>
+                <cylinder radius="0.02" length="0.01"/>
+            </geometry>
+        </collision>
+        <xacro:inertial_cylinder mass= "0.06" radius="0.02" length="0.01">
+            <origin xyz="0 0 0" rpy="0 0 0"/>
+        </xacro:inertial_cylinder>
     </link>
     <joint name="base_joint_b_R" type="fixed">
@@ -38,4 +55,12 @@
             <material name="gray"/>
         </visual>
+        <collision>
+            <geometry>
+                <cylinder radius="0.02" length="0.01"/>
+            </geometry>
+        </collision>
+        <xacro:inertial_cylinder mass= "0.06" radius="0.02" length="0.01">
+            <origin xyz="0 0 0" rpy="0 0 0"/>
+        </xacro:inertial_cylinder>
     </link>
     <joint name="base_joint__motor_pitch" type="fixed">
@@ -53,4 +78,12 @@
             <material name="blue"/>
         </visual>
+        <collision>
+            <geometry>
+                <cylinder radius="0.12" length="0.001"/>
+            </geometry>
+        </collision>
+        <xacro:inertial_cylinder mass= "0.02" radius="0.12" length="0.001">
+            <origin xyz="0 0 0" rpy="0 0 0"/>
+        </xacro:inertial_cylinder>
     </link>
     <joint name="rotor_l_joint" type="continuous">
@@ -68,4 +101,12 @@
             <material name="blue"/>
         </visual>
+        <collision>
+            <geometry>
+                <cylinder radius="0.12" length="0.001"/>
+            </geometry>
+        </collision>
+        <xacro:inertial_cylinder mass= "0.02" radius="0.12" length="0.001">
+            <origin xyz="0 0 0" rpy="0 0 0"/>
+        </xacro:inertial_cylinder>
     </link>
     <joint name="rotor_r_joint" type="continuous">
@@ -83,4 +124,12 @@
             <material name="blue"/>
         </visual>
+        <collision>
+            <geometry>
+                <cylinder radius="0.12" length="0.001"/>
+            </geometry>
+        </collision>
+        <xacro:inertial_cylinder mass= "0.02" radius="0.12" length="0.001">
+            <origin xyz="0 0 0" rpy="0 0 0"/>
+        </xacro:inertial_cylinder>
     </link>
     <joint name="rotor_pitch_joint" type="continuous">

File: description/camera.xacro (robot description, xacro)
@@ -4,5 +4,5 @@
         <parent link="u_shape_base_link"/>
         <child link="camera_link"/>
-        <origin xyz="-0.02 0.0 -0.01" rpy="0.0 0.0 0.0"/>
+        <origin xyz="-0.02 0.0 -0.01" rpy="0 ${pi/2} 0.0"/>
     </joint>
     <link name="camera_link">
@@ -11,11 +11,19 @@
                 <box size="0.023 0.023 0.005"/>
             </geometry>
+            <material name="red"/>
         </visual>
-        <material name="red"/>
+        <collision>
+            <geometry>
+                <box size="0.023 0.023 0.005"/>
+            </geometry>
+        </collision>
+        <xacro:inertial_box mass= "0.001" x="0.023" y="0.023" z="0.005">
+            <origin xyz="0 0 0" rpy="0 0 0"/>
+        </xacro:inertial_box>
     </link>
     <joint name="camera_optical_joint" type="fixed">
         <parent link="camera_link"/>
         <child link="camera_link_optical"/>
-        <origin xyz="0 0 0" rpy="${-pi/2} 0.0 ${-pi/2}"/>
+        <origin xyz="0 0 0" rpy="0.0 ${pi/2} 0.0"/>
     </joint>
     <link name="camera_link_optical">
@@ -29,4 +37,5 @@
             <camera>
                 <horizontal_fov>1.089</horizontal_fov>
+                <vertical_fov>1.089</vertical_fov>
                 <image>
                     <format>R8G8B8</format>
@@ -39,5 +48,5 @@
                 </clip>
             </camera>
-            <plugin name="camera_controller" filename="libgazebo_ros_cmaera.so">
+            <plugin name="camera_controller" filename="libgazebo_ros_camera.so">
                 <frame_name>camera_link_optical</frame_name>
             </plugin>

File: description/robot.urdf.xacro (robot description, xacro)
@@ -4,3 +4,5 @@
     <xacro:include filename="robot_core.xacro"/>
     <xacro:include filename="bldc_motor.xacro"/>
+    <xacro:include filename="imu.xacro"/>
+    <xacro:include filename="camera.xacro"/>
 </robot>

File: description/robot_core.xacro (robot description, xacro)
@@ -1,4 +1,5 @@
 <?xml version="1.0"?>
 <robot xmlns:xacro="http://www.ros.org/wiki/xacro" >
+    <xacro:include filename="inertial_macros.xacro"/>
     <material name="white">
         <color rgba="1.0 1.0 1.0 1.0"/>
@@ -12,4 +13,7 @@
     <material name="blue">
         <color rgba="0.0 0.0 1.0 0.5"/>
+    </material>
+    <material name="red">
+        <color rgba="1 0 0 1"/>
     </material>
     <link name="base_link">
@@ -28,6 +32,18 @@
             <material name="white"/>
         </visual>
-    </link>
-    <!-- Hinge Support -->
+        <collision>
+            <geometry>
+                <cylinder radius="0.091" length="0.0182"/>
+            </geometry>
+        </collision>
+        <xacro:inertial_cylinder mass = "1.278403083" length="0.0182" radius="0.091">
+            <origin xyz = "0 0 0" rpy = "0 0 0"/>
+        </xacro:inertial_cylinder>
+    </link>
+    <gazebo reference="base_plate_link">
+        <material>Gazebo/White</material>
+    </gazebo>
+    <!-- Base Plate Done -->
+    <!-- Vertical Rod Support -->
     <joint name="support_base_joint" type="fixed">
         <origin xyz="0.0 0.0 0.16" rpy="0.0 0.0 0.0"/>
@@ -43,5 +59,17 @@
             <material name="white"/>
         </visual>
-    </link>
+        <collision>
+            <geometry>
+                <cylinder radius="0.011" length="0.32"/>
+            </geometry>
+        </collision>
+        <xacro:inertial_cylinder mass = "0.328434662377" length="0.32" radius="0.091">
+            <origin xyz="0.0 0.0 0.0" rpy="0.0 0.0 0.0"/>
+        </xacro:inertial_cylinder>
+    </link>
+    <gazebo reference="support_base_link">
+        <material>Gazebo/White</material>
+    </gazebo>
+    <!-- Vertical Rod is done -->
     <!-- U shape base -->
     <joint name="u_shape_base" type="continuous">
@@ -59,5 +87,16 @@
             <material name="white"/>
         </visual>
-    </link>
+        <collision>
+            <geometry>
+                <box size="0.05 0.05 0.015"/>
+            </geometry>
+        </collision>
+        <xacro:inertial_box mass= "0.10125" x="0.05" y="0.05" z="0.015">
+            <origin xyz="0 0 0" rpy="0 0 0"/>
+        </xacro:inertial_box>
+    </link>
+    <gazebo reference="u_shape_base_link">
+        <material>Gazebo/White</material>
+    </gazebo>
     <!-- U Shape Pillars -->
     <joint name="u_shape_pillar_r_joint" type="fixed">
@@ -74,5 +113,17 @@
             <material name="white"/>
         </visual>
-    </link>
+        <collision>
+            <origin xyz="0.0 0.0 0.03" rpy="0.0 0.0 0.0"/>
+            <geometry>
+                <box size="0.01 0.05 0.06"/>
+            </geometry>
+        </collision>
+        <xacro:inertial_box mass= "0.081" x="0.01" y="0.05" z="0.06">
+            <origin xyz="0 0 0.3" rpy="0 0 0"/>
+        </xacro:inertial_box>
+    </link>
+    <gazebo reference="u_shape_pillar_r_link">
+        <material>Gazebo/White</material>
+    </gazebo>
     <joint name="u_shape_pillar_l_joint" type="fixed">
         <parent link="u_shape_base_link"/>
@@ -88,5 +139,18 @@
             <material name="white"/>
         </visual>
-    </link>
+        <collision>
+            <origin xyz="0.0 0.0 0.03" rpy="0.0 0.0 0.0"/>
+            <geometry>
+                <box size="0.01 0.05 0.06"/>
+            </geometry>
+        </collision>
+        <xacro:inertial_box mass= "0.081" x="0.01" y="0.05" z="0.06">
+            <origin xyz="0 0 0.3" rpy="0 0 0"/>
+        </xacro:inertial_box>
+    </link>
+    <gazebo reference="u_shape_pillar_l_link">
+        <material>Gazebo/White</material>
+    </gazebo>
+    <!-- pillars and fork done -->
     <!-- Pin Connecting both pillars -->
     <joint name="pillar_connecting_joint" type="fixed">
@@ -103,5 +167,17 @@
             <material name="white"/>
         </visual>
-    </link>
+        <collision>
+            <geometry>
+                <cylinder radius="0.0075" length="0.05"/>
+            </geometry>
+        </collision>
+        <xacro:inertial_cylinder mass= "0.023856469" radius="0.0075" length="0.05">
+            <origin xyz="0 0 0.0" rpy="0 0 0"/>
+        </xacro:inertial_cylinder>
+    </link>
+    <gazebo reference="pillar_connecting_link">
+        <material>Gazebo/White</material>
+    </gazebo>
+    <!-- Connecting Pin Done -->
     <!-- Hinge at the Pin -->
     <joint name="pin_hinge_joint" type="revolute">
@@ -120,5 +196,16 @@
             <material name="white"/>
         </visual>
-    </link>
+        <collision>
+            <geometry>
+                <box size="0.02 0.02 0.04"/>
+            </geometry>
+        </collision>
+        <xacro:inertial_box mass= "0.0432" x="0.02" y="0.02" z="0.04">
+            <origin xyz="0 0 0" rpy="0 0 0"/>
+        </xacro:inertial_box>
+    </link>
+    <gazebo reference="pin_hinge_link">
+        <material>Gazebo/White</material>
+    </gazebo>
     <!-- Main Beam Link -->
     <joint name="beam_joint" type="fixed">
@@ -135,4 +222,15 @@
             <material name="black"/>
         </visual>
-    </link>
+        <collision>
+            <geometry>
+                <box size="0.012 0.55 0.012"/>
+            </geometry>
+        </collision>
+        <xacro:inertial_box mass= "0.21384" x="0.012" y="0.55" z="0.012">
+            <origin xyz="0 0 0" rpy="0 0 0"/>
+        </xacro:inertial_box>
+    </link>
+    <gazebo reference="beam_link">
+        <material>Gazebo/Black</material>
+    </gazebo>
 </robot>
