Commit message: commit

File: description/imu.xacro (robot description, xacro)
@@ -13,26 +13,4 @@
             <material name="red"/>
         </visual>
-        <collision>
-            <geometry>
-                <box size="0.01 0.047 0.035"/>
-            </geometry>
-        </collision>
-        <xacro:inertial_box mass= "0.001" x="0.01" y="0.047" z="0.035">
-            <origin xyz="0 0 0" rpy="0 0 0"/>
-        </xacro:inertial_box>
     </link>
-    <gazebo reference="imu_link">
-        <material>Gazebo/Red</material>
-        <sensor name="my_imu" type="imu">
-            <always_on>true</always_on>
-            <update_rate>30</update_rate>
-            <plugin name="my_imu_plugin" filename="libgazebo_ros_imu_sensor.so">
-                <ros>
-                    <namespace>imu</namespace>
-                    <remapping>~/out:=data</remapping>
-                </ros>
-                <frame_name>imu_link</frame_name>
-            </plugin>
-        </sensor>
-    </gazebo>
 </robot>
